Commit message: feat: K1_locomotion.urdfをモデルとして利用するように変更

File: assets_soccer/booster_robotics_robots/K1/K1_locomotion.urdf (robot description, URDF)
Before this commit: robot K1, 23 links, 22 joints
Joints:
- joint Left_Shoulder_Roll: origin xyz=0.0025 0.068 -0.0135 rpy=0 0 0 -> xyz=0.0025 0.068 -0.0135 rpy=-1.3744467860 0 0
- joint Right_Shoulder_Roll: origin xyz=0.0025 -0.068 -0.0135 rpy=0 0 0 -> xyz=0.0025 -0.068 -0.0135 rpy=1.3744467860 0 0
