Commit message: fix: K1 の Hip_Pitch 寸法を修正し、足裏スピン抵抗入り USD を生成して使う
## URDF の寸法修正

Hip_Pitch 関節原点の z を -0.077 → -0.062 に修正 (左右 2 箇所)。
NOTE: 同じ値が ARight_Shoulder_Pitch の **y 成分** にも出現するが、そちらは
肩関節で無関係なので変更していない (一括置換は不可)。

## 足裏のトーショナル摩擦 (スピン抵抗)

実機・MuJoCo では足裏が地面をスピンする際にトーショナル摩擦が抵抗トルクを生むが、
IsaacLab の通常の設定経路では K1 に適用できなかった:

  1. startup イベントで複製後の prim に modify_collision_properties
     → 失敗。env は USD インスタンスとして複製されるため個別編集不可
       (4096 prim 全てで "instanced prim" 警告)
  2. spawn の collision_props に設定 (複製前に効かせる狙い)
     → 失敗。URDF→USD 変換が各リンクの collisions prim を既にインスタンス化済みで、
       env_0 の時点で編集できない
  3. AssetConverterBaseCfg.make_instanceable=False
     → 無効。urdf_converter.py はこのフラグを一度も参照せず instanceable 固定
       (docstring にも "stores the output USD file in an instanceable format" と明記)

結果として Isaac 内では足裏が実質無抵抗でスピンでき、その場回転タスクの方策は
「接地したまま捻る」戦略に居座っていた。摩擦係数の DR は並進の滑りにしか効かないため、
平均 0.82→1.65 に上げても踏み替えは一切獲得されなかった (片足支持時間 0.0040→0.0037)。
その帰結が sim2sim ギャップで、Isaac で成功率 97.7% の 130-180° が MuJoCo では
ほとんど失敗し、破綻率は必要スピン量に比例して増えていた
(0-50°: 0.3% / 50-90°: 0.4% / 90-130°: 0.9% / 130-180°: 2.0%)。

## make_k1_usd_torsional.py

変換後の configuration/K1_locomotion_physics.usd を単体で開くと足の collision prim は
インスタンス化されていないため編集できる。ここに PhysxCollisionAPI を適用して
torsionalPatchRadius=0.04 (MuJoCo の足 box 0.18x0.07 m 相当) を書き込む。

生成物 assets_soccer/booster_robotics_robots/K1/usd_torsional/ を K1FlatTurnCfg が
UsdFileCfg で読む。K1_LOCOMOTION_CFG はモジュール共有なので、他タスク (歩行 /
dribble / kick) に影響しないよう本タスクのコピーに対してのみ差し替えている。

検証済み:
  * torsionalPatchRadius が足 2 prim のみに入る (CollisionAPI 20 個中)
  * Hip_Pitch の localPos0 = (0, ±0.096, -0.062) と修正が反映されている
  * 可動関節 12 個が JOINT_NAMES_K1 と完全一致 (観測 49 次元レイアウトは不変)
  * env 側の spawn が UsdFileCfg で当該 USD を指し、URDF 変換が走らない

NOTE: この USD は URDF のスナップショット。URDF を変更したらスクリプトの再実行が必要。
NOTE: 既存の学習済みポリシーは全て旧寸法 (-0.077) で学習されているため、
      本コミット以降は warm-start の起点として使えない。

Co-Authored-By: Claude Opus 5 (1M context) <noreply@anthropic.com>
Claude-Session: https://claude.ai/code/session_01UE4Y8m1HWh9e2pDmQ39Ng9

File: assets_soccer/booster_robotics_robots/K1/K1_locomotion.urdf (robot description, URDF)
Before this commit: robot K1, 23 links, 22 joints
Joints:
- joint Left_Hip_Pitch: origin xyz=0 0.096 -0.077 rpy=0 0 0 -> xyz=0 0.096 -0.062 rpy=0 0 0
- joint Right_Hip_Pitch: origin xyz=0 -0.096 -0.077 rpy=0 0 0 -> xyz=0 -0.096 -0.062 rpy=0 0 0
